File: i2c_esc/KiCad/ESC/esc.kicad_pcb (KiCad board)
At the start: 2 copper layers, 11 parts, among them J1 ESC_1, J2 ESC_2, J3 ESC_3, J4 ESC_4, J5 I2C_Bus, J6 icsp, U1 ATMEGA328P-AU, Y1 Crystal_GND3

Commit message: pcb update
Parts:
- added C2: C, Capacitors_SMD:C_0603, F.Cu at (124.0, 92.5)
- added C3: C, Capacitors_SMD:C_0603, F.Cu at (124.0, 75.7)
- added J7: Conn_01x02, Pin_Headers:Pin_Header_Angled_1x02_Pitch2.00mm, F.Cu at (143.8, 81.8)
- C1: footprint Crystals:Crystal_SMD_EuroQuartz_EQ161-2pin_3.2x1.5mm -> Capacitors_SMD:C_0603
- J1, J2, J3, J4: footprint Pin_Headers:Pin_Header_Angled_1x03_Pitch1.00mm -> Pin_Headers:Pin_Header_Angled_1x03_Pitch2.00mm
- J5: footprint Pin_Headers:Pin_Header_Angled_1x02_Pitch1.00mm -> Pin_Headers:Pin_Header_Angled_1x02_Pitch2.00mm
- J6: footprint Pin_Headers:Pin_Header_Straight_2x03_Pitch1.00mm_SMD -> Pin_Headers:Pin_Header_Straight_2x03_Pitch2.00mm
- JP1: footprint Pin_Headers:Pin_Header_Straight_1x02_Pitch1.00mm_SMD_Pin1Left -> Pin_Headers:Pin_Header_Straight_1x02_Pitch2.00mm
- R1: footprint Resistors_SMD:R_0402 -> Resistors_SMD:R_0805
- Y1: value Crystal_GND3 -> Crystal; footprint Crystals:Crystal_SMD_0603-2pin_6.0x3.5mm -> Crystals:Crystal_SMD_HC49-SD
- moved J1 53.0 mm to (124.0, 72.6), turned to 180 degrees
- moved J4 50.5 mm to (143.8, 68.6)
- moved J2 41.3 mm to (124.0, 99.6), turned to 180 degrees
- moved J5 39.5 mm to (132.6, 74.2), turned to 90 degrees
- moved Y1 35.5 mm to (124.0, 84.3), turned to 90 degrees
- moved U1 34.4 mm to (133.1, 84.3)
- moved C1 29.5 mm to (140.7, 84.3), turned to 90 degrees
- moved JP1 16.7 mm to (118.4, 82.5), turned to 180 degrees
- moved J3 9.08 mm to (143.8, 95.5)
- moved J6 7.89 mm to (136.1, 96.0), turned to 270 degrees
- moved R1 4.33 mm to (118.4, 88.4), turned to 90 degrees
Connections:
- U1 pad 27: Net-(J5-Pad1) -> Net-(J5-Pad2)
- U1 pad 28: Net-(J5-Pad2) -> Net-(J5-Pad1)
Routing:
- net VCC: track 0.00 -> 57.6 mm, vias 0 -> 4
- net ESC_4_PWM: track 0.00 -> 46.0 mm
- net GND: track 0.00 -> 22.7 mm, vias 0 -> 2
- net Net-(JP1-Pad1): track 0.00 -> 20.9 mm, vias 0 -> 2
- net Net-(J6-Pad4): track 0.00 -> 20.9 mm, vias 0 -> 1
- net Net-(J6-Pad5): track 0.00 -> 20.1 mm, vias 0 -> 1
- net ESC_3_PWM: track 0.00 -> 17.8 mm
- net ESC_2_PWM: track 0.00 -> 16.6 mm
- net Net-(J6-Pad3): track 0.00 -> 16.6 mm, vias 0 -> 1
- net Net-(C3-Pad1): track 0.00 -> 14.4 mm
- net ESC_1_PWM: track 0.00 -> 12.4 mm
- net Net-(C2-Pad1): track 0.00 -> 9.68 mm
- net Net-(J6-Pad1): track 0.00 -> 7.57 mm, vias 0 -> 1
- net Net-(J5-Pad1): track 0.00 -> 6.29 mm
- net Net-(J5-Pad2): track 0.00 -> 6.03 mm
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- added copper zone on B.Cu, net GND
- added copper zone on F.Cu, net GND
Other:
- board outline added: 36 x 36 mm
- rule pad_to_mask_clearance: 0.2 -> 0
