File: i2c_esc/KiCad/ESC/esc.sch (KiCad schematic (older format))
At the start: 11 parts, among them J1 ESC_1, J2 ESC_2, J3 ESC_3, J4 ESC_4, J5 I2C_Bus, J6 icsp, U1 ATMEGA328P-AU, Y1 Crystal_GND3

Commit message: pcb update
Parts:
- removed Y1: Crystal_GND3, Crystals:Crystal_SMD_0603-2pin_6.0x3.5mm, symbol Crystal_GND3
- added C2, C3: C, Capacitors_SMD:C_0603, symbol C
- added J7: Conn_01x02, Pin_Headers:Pin_Header_Angled_1x02_Pitch2.00mm, symbol Conn_01x02
- added Y1: Crystal, Crystals:Crystal_SMD_HC49-SD, symbol Crystal
- C1: footprint Crystals:Crystal_SMD_EuroQuartz_EQ161-2pin_3.2x1.5mm -> Capacitors_SMD:C_0603
- J1, J2, J3, J4: footprint Pin_Headers:Pin_Header_Angled_1x03_Pitch1.00mm -> Pin_Headers:Pin_Header_Angled_1x03_Pitch2.00mm
- J5: footprint Pin_Headers:Pin_Header_Angled_1x02_Pitch1.00mm -> Pin_Headers:Pin_Header_Angled_1x02_Pitch2.00mm
- J6: footprint Pin_Headers:Pin_Header_Straight_2x03_Pitch1.00mm_SMD -> Pin_Headers:Pin_Header_Straight_2x03_Pitch2.00mm
- JP1: footprint Pin_Headers:Pin_Header_Straight_1x02_Pitch1.00mm_SMD_Pin1Left -> Pin_Headers:Pin_Header_Straight_1x02_Pitch2.00mm
- R1: footprint Resistors_SMD:R_0402 -> Resistors_SMD:R_0805
Connections:
- net GND: now also C2.2, C3.2, J7.2 (Pin_2)
- net VCC: now also J7.1 (Pin_1)
- net at U1.27 ((PCINT12/SDA/ADC4)PC4): now also J5.2 (Pin_2); no longer J5.1 (Pin_1)
- net at U1.28 ((PCINT13/SCL/ADC5)PC5): now also J5.1 (Pin_1); no longer J5.2 (Pin_2)
- net at U1.7 ((PCINT6/XTAL1/TOSC1)PB6): now also C3.1, Y1.2
- net at U1.8 ((PCINT7/XTAL2/TOSC2)PB7): now also C2.1, Y1.1
